File: Hardware/ESP32_C3_LVGL_DEVBOARD/ESP32_C3_LVGL_DEVBOARD.kicad_pcb (KiCad board)
At the start: 4 copper layers, 27 x 40 mm, 68 parts, among them J1 CONN_USBC, J2 CONN_UART, J3 Conn_Coaxial, SW1 SW_Push_SPST_4Pads, SW2 SW_Push_SPST_4Pads, U2 USBLC6-2SC6, U3 AMS1117-3.3, U4 ESP32-C3, U5 Winbond-W25Q64JVSSIQ, U6 USBLC6-2SC6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

Commit message: pcb committ
Routing:
- net GND: vias 127 -> 116
